File: _saved_Anti-Spark-Switch.sch (KiCad schematic (older format))
At the start: 12 parts, among them P2 Pad_Conn, P5 Pad_Conn, P6 Pad_Conn, P7 CONN_01X02, Q1 IRFS7530, Q2 IRFS7530, Q3 IRFS7530

Commit message: smaller design
Parts:
- removed P7: CONN_01X02, Connector_JST:JST_PH_B4B-PH-K_1x02_P2.00mm_Vertical, symbol conn:Conn_01x02
- C1: footprint Capacitors_SMD:C_0603 -> Capacitor_SMD:C_0805_2012Metric_Pad1.33x1.40mm_HandSolder
- D1: footprint Diodes_SMD:D_SOD-123F -> Diode_SMD:D_SOD-123F
- P5: value Pad_Conn -> VCC NO
- P6: value Pad_Conn -> OUT -
- R1, R2, R3: footprint Resistors_SMD:R_0603 -> Resistor_SMD:R_0805_2012Metric_Pad1.33x1.40mm_HandSolder
Connections:
- net labels removed: VCC
- wire segments 41 -> 36
Other:
- moved on the sheet: P5
Changed lines of the file:
@@
 F 0 "R2" V 4730 4050 50  0000 C CNN
 F 1 "1M" V 4650 4050 50  0000 C CNN
-F 2 "Resistors_SMD:R_0603" V 4580 4050 50  0001 C CNN
+F 2 "Resistor_SMD:R_0805_2012Metric_Pad1.33x1.40mm_HandSolder" V 4580 4050 50  0001 C CNN
 F 3 "" H 4650 4050 50  0000 C CNN
 	1    4650 4050
@@
 F 0 "R3" V 5430 3350 50  0000 C CNN
 F 1 "1K" V 5350 3350 50  0000 C CNN
-F 2 "Resistors_SMD:R_0603" V 5280 3350 50  0001 C CNN
+F 2 "Resistor_SMD:R_0805_2012Metric_Pad1.33x1.40mm_HandSolder" V 5280 3350 50  0001 C CNN
 F 3 "" H 5350 3350 50  0000 C CNN
 	1    5350 3350
@@
 F 0 "C1" H 5075 3650 50  0000 L CNN
 F 1 "1uF" H 5075 3450 50  0000 L CNN
-F 2 "Capacitors_SMD:C_0603" H 5088 3400 50  0001 C CNN
+F 2 "Capacitor_SMD:C_0805_2012Metric_Pad1.33x1.40mm_HandSolder" H 5088 3400 50  0001 C CNN
 F 3 "" H 5050 3550 50  0000 C CNN
 	1    5050 3550
@@
 F 0 "D1" H 5050 4250 50  0000 C CNN
 F 1 "ZENER" H 5050 4050 50  0000 C CNN
-F 2 "Diodes_SMD:D_SOD-123F" H 5050 4150 50  0001 C CNN
+F 2 "Diode_SMD:D_SOD-123F" H 5050 4150 50  0001 C CNN
 F 3 "" H 5050 4150 50  0000 C CNN
 	1    5050 4150
@@
 F 3 "" H 4100 4600 50  0000 C CNN
 	1    4100 4600
-	1    0    0    -1
-$EndComp
-$Comp
-L power:VCC #PWR02
-U 1 1 5775E532
-P 7650 2900
-F 0 "#PWR02" H 7650 2750 50  0001 C CNN
-F 1 "VCC" H 7650 3050 50  0000 C CNN
-F 2 "" H 7650 2900 50  0000 C CNN
-F 3 "" H 7650 2900 50  0000 C CNN
-	1    7650 2900
 	1    0    0    -1
 $EndComp
@@
 P 7950 3350
 F 0 "P6" H 7950 3450 50  0000 C CNN
-F 1 "Pad_Conn" H 8050 3250 50  0000 C CNN
+F 1 "OUT -" H 8050 3250 50  0000 C CNN
 F 2 "sparkparts:1PAD_8x7mm" V 7950 3350 50  0001 C CNN
 F 3 "" H 7950 3350 50  0000 C CNN
 	1    7950 3350
-	1    0    0    -1
-$EndComp
-$Comp
-L Anti-Spark-Switch-rescue:Pad_Conn P5
-U 1 1 577ED9DE
-P 7950 3050
-F 0 "P5" H 7950 3150 50  0000 C CNN
-F 1 "Pad_Conn" H 8050 2950 50  0000 C CNN
-F 2 "Connector_PinHeader_2.54mm:PinHeader_1x01_P2.54mm_Vertical" H 7950 3050 50  0001 C CNN
-F 3 "" H 7950 3050 50  0000 C CNN
-	1    7950 3050
 	1    0    0    -1
 $EndComp
@@
 $EndComp
 Wire Wire Line
-	7650 3050 7650 2900
-Wire Wire Line
 	4100 4600 4100 4450
 Wire Wire Line
@@
 Wire Wire Line
 	3900 4450 4100 4450
-Connection ~ 7650 3050
 Wire Wire Line
 	4650 3750 5050 3750
@@
 Wire Wire Line
 	6000 3350 6700 3350
-Wire Wire Line
-	7650 3050 7750 3050
-$Comp
-L conn:Conn_01x02 P7
-U 1 1 577ECAA0
-P 4350 3650
-F 0 "P7" H 4350 3850 50  0000 C CNN
-F 1 "CONN_01X02" V 4450 3650 50  0000 C CNN
-F 2 "Connector_JST:JST_PH_B4B-PH-K_1x02_P2.00mm_Vertical" H 4350 3650 50  0001 C CNN
-F 3 "" H 4350 3650 50  0000 C CNN
-	1    4350 3650
-	-1   0    0    1
-$EndComp
 Wire Wire Line
 	4100 4450 4650 4450
@@
 L device:R R1
 U 1 1 5775E3D7
-P 4650 3300
-F 0 "R1" V 4730 3300 50  0000 C CNN
-F 1 "1M" V 4650 3300 50  0000 C CNN
-F 2 "Resistors_SMD:R_0603" V 4580 3300 50  0001 C CNN
-F 3 "" H 4650 3300 50  0000 C CNN
-	1    4650 3300
-	1    0    0    -1
-$EndComp
-Wire Wire Line
-	4650 3050 4650 3150
-Wire Wire Line
-	4650 3450 4650 3550
-Wire Wire Line
-	4650 3550 4550 3550
-Wire Wire Line
-	4550 3650 4650 3650
-Wire Wire Line
-	4650 3650 4650 3750
+P 4650 3450
+F 0 "R1" V 4730 3450 50  0000 C CNN
+F 1 "1M" V 4650 3450 50  0000 C CNN
+F 2 "Resistor_SMD:R_0805_2012Metric_Pad1.33x1.40mm_HandSolder" V 4580 3450 50  0001 C CNN
+F 3 "" H 4650 3450 50  0000 C CNN
+	1    4650 3450
+	1    0    0    -1
+$EndComp
+Wire Wire Line
+	7400 3350 7750 3350
+Wire Wire Line
+	6900 3350 7400 3350
+Wire Wire Line
+	6700 3350 7400 3350
+Wire Wire Line
+	4650 3600 4650 3750
 Connection ~ 4650 3750
-Wire Wire Line
-	4650 3050 7650 3050
-Wire Wire Line
-	7400 3350 7750 3350
-Wire Wire Line
-	6900 3350 7400 3350
-Wire Wire Line
-	6700 3350 7400 3350
+$Comp
+L Anti-Spark-Switch-rescue:Pad_Conn P5
+U 1 1 577ED9DE
+P 4350 3200
+F 0 "P5" H 4269 2975 50  0000 C CNN
+F 1 "VCC NO" H 4269 3066 50  0000 C CNN
+F 2 "Connector_PinHeader_2.54mm:PinHeader_1x01_P2.54mm_Vertical" H 4350 3200 50  0001 C CNN
+F 3 "" H 4350 3200 50  0000 C CNN
+	1    4350 3200
+	-1   0    0    1
+$EndComp
+Wire Wire Line
+	4550 3200 4650 3200
+Wire Wire Line
+	4650 3200 4650 3300
 $EndSCHEMATC
